File: SimpleServoTester/SimpleServoTester.kicad_sch (KiCad schematic)
At the start: 8 parts, among them SW1 POWER, U1 ATmega328-A, U2 L7805

Commit message: update
Parts:
- added C10, C11, C14, C15, C4, C5, C6, C9: 100n/50V, symbol Device:C_Small
- added C12, C13: 10uF/50V, symbol Device:C_Polarized_Small
- added D1: 1N4001, symbol Device:D_Small
- added H1, H2, H3, H4: MountingHole, symbol Mechanical:MountingHole
- added J2: Servo, symbol Connector:Conn_01x03_Pin
- added J2: USBASP, Connector_IDC:IDC-Header_2x05_P2.54mm_Horizontal, symbol Connector_Generic:Conn_02x05_Odd_Even
- added J3: OLED, symbol Connector:Conn_01x04_Socket
- added L1: 10u, symbol Device:L_Small
- added Q1: IRLZ44N, Package_TO_SOT_THT:TO-220-3_Vertical, symbol Transistor_FET:IRLZ44N
- added R2, R3, R4, R5, R6: 10k, symbol Device:R_Small
- added R7: 0.1R, symbol Device:R_Shunt
- added R9: 100R, symbol Device:R_Small
- added RV1: 10k, symbol Device:R_Potentiometer
- added SW2: Tactile, symbol Switch:SW_MEC_5E
- added U3: INA219AxD, Package_SO:SOIC-8_3.9x4.9mm_P1.27mm, symbol Sensor_Energy:INA219AxD
- added U4: AMS1117-3.3, Package_TO_SOT_SMD:SOT-223-3_TabPin2, symbol Regulator_Linear:AMS1117-3.3
- added Y2: 16MHz, Footprint:CSTCE16M0V53-R0, symbol Device:Resonator_Small
Connections:
- net +5V: now also U1.20 (AREF), U1.4 (VCC), U1.6 (VCC), C4.1, C6.1, C9.1, D1.1 (K), L1.2, R3.1, R4.1, R7.1, RV1.3, U3.5 (VS)
- net GND: now also C10.2, C11.2, C12.2, C13.2, C14.2, C15.1, C4.2, C5.2, C6.2, C9.2, J2.10 (Pin_10), J2.4 (Pin_4), J2.6 (Pin_6), J2.8 (Pin_8), J3.4 (Pin_4), Q1.3 (S), R2.2, R5.2, R6.2, RV1.1, SW2.1, SW2.2, U3.6 (GND), U4.1 (GND), Y2.2
- net +BATT: now reaches C1.1, SW1.2 (B), U2.1 (IN)
- net +BATT: now also C11.1, C13.1, U4.3 (VI)
- net SERVO_SIGNAL: now reaches U1.13 (PB1)
- net SERVO_SIGNAL: now also J2.3 (Pin_3)
- net MOSI: now reaches U1.15 (PB3)
- net MOSI: now also J2.1 (Pin_1)
- net MISO: now reaches U1.16 (PB4)
- net MISO: now also J2.9 (Pin_9)
- net SCK: now reaches U1.17 (PB5)
- net SCK: now also J2.7 (Pin_7)
- net at U1.18 (AVCC): now also C5.1, L1.1
- net POT: now reaches U1.23 (PC0)
- net POT: now also C10.1, RV1.2
- net SDA: now reaches U1.27 (PC4)
- net SDA: now also J3.1 (Pin_1), R3.2, U3.3 (SDA)
- net SCL: now reaches U1.28 (PC5)
- net SCL: now also J3.2 (Pin_2), R4.2, U3.4 (SCL)
- net RESET: now reaches R1.2, U1.29 (~{RESET}/PC6)
- net RESET: now also J2.5 (Pin_5)
- net GATE_MOSFET: now reaches U1.30 (PD0)
- net GATE_MOSFET: now also Q1.1 (G), R2.1
- net INT_PIN: now reaches U1.32 (PD2)
- net INT_PIN: now also C15.2, R9.2
- net at U1.7 (XTAL1/PB6): now also Y2.3
- net at U1.8 (XTAL2/PB7): now also Y2.1
- new net: R6.1, U3.1 (A1)
- new net: J2.1 (Pin_1), Q1.2 (D)
- new net: D1.2 (A), J2.2 (Pin_2)
- new net: J2.2 (Pin_2), R7.4
- new net: R9.1, SW2.3 (K), SW2.4 (A)
- new net: R5.1, U3.2 (A0)
- new net: R7.3, U3.7 (IN-)
- new net: R7.2, U3.8 (IN+)
- new net +3V3: C12.1, C14.1, J3.3 (Pin_3), U4.2 (VO)
- no-connect marks 0 -> 14
Other:
- note added: "BAT > 3V3"
- note added: "BAT > 5V"
- note added: "I2C PULLUP"
- note added: "MECHANICAL"
- note added: "MICROCONTROLLER"
- note added: "MOSFET / SERVO / CURRENT SENSE"
- note added: "OLED"
- note added: "POTENTIOMETER"
- note added: "PROGRAM PORT"
- note added: "TACTILE"
- note added: "USBASP"
- moved on the sheet: BT1, C1, C2, C3, R1, SW1, U1, U2

Commit message: update
Parts:
- removed BT1: 2x18650, symbol Device:Battery
- removed R7: 0.1R, symbol Device:R_Shunt
- removed SW2: Tactile, symbol Switch:SW_MEC_5E
- removed U2: L7805, symbol Regulator_Linear:L7805
- added BT1, BT2: Battery_Cell, Footprint:18650-PC2, symbol Device:Battery_Cell
- added R7: 0.1R, Resistor_SMD:R_0603_1608Metric, symbol Device:R_Small
- added SW2: RotaryEncoder_Switch, symbol Device:RotaryEncoder_Switch
- added U2: LM7805_TO220, Package_TO_SOT_THT:TO-220-3_Horizontal_TabDown, symbol Regulator_Linear:LM7805_TO220
- C1, C12, C13, C3: footprint (none) -> Capacitor_SMD:CP_Elec_5x5.4
- C10, C11, C14, C15, C2, C4, C5, C6, C9: footprint (none) -> Capacitor_SMD:C_0603_1608Metric
- D1: footprint (none) -> Diode_SMD:D_SMA
- H1, H2, H3, H4: footprint (none) -> MountingHole:MountingHole_3.2mm_M3_Pad_Via
- J2: footprint (none) -> Connector_PinHeader_2.54mm:PinHeader_1x03_P2.54mm_Horizontal
- J3: footprint (none) -> Connector_PinSocket_2.54mm:PinSocket_1x04_P2.54mm_Vertical
- L1: footprint (none) -> Inductor_SMD:L_1206_3216Metric
- Q1: footprint Package_TO_SOT_THT:TO-220-3_Vertical -> Package_TO_SOT_THT:TO-220-3_Horizontal_TabDown
- R1, R2, R3, R4, R5, R6, R9: footprint (none) -> Resistor_SMD:R_0603_1608Metric
- RV1: footprint (none) -> Footprint:PTV09A-4225F-B502
- SW1: footprint (none) -> Connector_PinHeader_2.54mm:PinHeader_1x02_P2.54mm_Vertical
- U3: footprint Package_SO:SOIC-8_3.9x4.9mm_P1.27mm -> Package_TO_SOT_SMD:SOT-23-8
Connections:
- net +5V: now also U3.8 (IN+), R7.1, U2.3 (VO)
- net +BATT: now also U2.1 (VI)
- net GND: now also BT2.2 (-), SW2.S2, U2.2 (GND)
- net at J2.2 (Pin_2): now also U3.7 (IN-), R7.2
- net S+: now reaches SW1.1 (A)
- net S+: now also BT1.1 (+)
- net VDD: now reaches C5.1, L1.1, U1.18 (AVCC)
- net at R9.1: now also SW2.S1
- new net: BT1.2 (-), BT2.1 (+)
Other:
- moved on the sheet: C15, R9

Commit message: update
Parts:
- removed C10: 100n/50V, Capacitor_SMD:C_0603_1608Metric, symbol Device:C_Small
- removed RV1: 10k, Footprint:PTV09A-4225F-B502, symbol Device:R_Potentiometer
- added C7, C8: 100n/50V, Capacitor_SMD:C_0603_1608Metric, symbol Device:C_Small
- added R10, R8: 100R, Resistor_SMD:R_0603_1608Metric, symbol Device:R_Small
- H1, H2, H3, H4: footprint MountingHole:MountingHole_3.2mm_M3_Pad_Via -> MountingHole:MountingHole_3.2mm_M3
- SW2: footprint (none) -> Rotary_Encoder:RotaryEncoder_Alps_EC11E-Switch_Vertical_H20mm
Connections:
- net GND: now also SW2.C, C7.1, C8.2
- net at SW2.A: now also R8.2
- net at SW2.B: now also R10.2
- net INT_PIN_2: now reaches U1.1 (PD3)
- net INT_PIN_2: now also C7.2, R8.1
- net DI: now reaches U1.2 (PD4)
- net DI: now also C8.1, R10.1
- no-connect marks 14 -> 12
Other:
- note removed: "POTENTIOMETER"
- moved on the sheet: C15, R9, SW2

Commit message: update
Parts:
- added Q2: S8050, Package_TO_SOT_SMD:SOT-23-3, symbol Transistor_BJT:S8050
- added R11: 1k, Resistor_SMD:R_0603_1608Metric, symbol Device:R_Small
- added R12, R13: 47k, Resistor_SMD:R_0603_1608Metric, symbol Device:R_Small
- R7: footprint Resistor_SMD:R_0603_1608Metric -> Resistor_SMD:R_2512_6332Metric
Connections:
- net POT is gone; now on net AI0: U1.23 (PC0)
- net +BATT: now also R13.1
- net GND: now also Q2.1 (E)
- net AI0: now reaches BT1.2 (-), BT2.1 (+)
- net BAT_T: now reaches U1.11 (PD7)
- net BAT_T: now also R11.1
- net AI1: now reaches U1.24 (PC1)
- net AI1: now also R12.1, R13.2
- new net: Q2.2 (B), R11.2
- new net: Q2.3 (C), R12.2
- no-connect marks 12 -> 9
Other:
- moved on the sheet: BT2

Commit message: update
Parts:
- removed J2: USBASP, Connector_IDC:IDC-Header_2x05_P2.54mm_Horizontal, symbol Connector_Generic:Conn_02x05_Odd_Even
- added J1: USBASP, Connector_PinHeader_2.54mm:PinHeader_1x06_P2.54mm_Horizontal, symbol Connector:Conn_01x06_Pin
Connections:
- net BAT_T: now also U1.25 (PC2); no longer U1.11 (PD7)
- net DI: now also U1.12 (PB0); no longer U1.2 (PD4)
- net GATE_MOSFET: now also U1.2 (PD4); no longer U1.30 (PD0)
- net GND: now also J1.6 (Pin_6)
- net INT_PIN: now also C7.2, R8.1; no longer C15.2, R9.2
- net INT_PIN_2: now also C15.2, R9.2; no longer C7.2, R8.1
- net MISO: now also J1.3 (Pin_3)
- net MOSI: now also J1.4 (Pin_4)
- net RESET: now also J1.5 (Pin_5)
- net SCK: now also J1.2 (Pin_2)
- net at D1.2 (A): now also J1.1 (Pin_1)
Other:
- note removed: "USBASP"
- moved on the sheet: D1

Commit message: update
Parts:
- J3: footprint Connector_PinSocket_2.54mm:PinSocket_1x04_P2.54mm_Vertical -> Connector_PinHeader_2.54mm:PinHeader_1x04_P2.54mm_Vertical
Changed lines of the file:
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@@
       (effects (font (size 1.27 1.27)) (justify left))
     )
-    (property "Footprint" "Connector_PinSocket_2.54mm:PinSocket_1x04_P2.54mm_Vertical" (at 218.44 34.29 0)
+    (property "Footprint" "Connector_PinHeader_2.54mm:PinHeader_1x04_P2.54mm_Vertical" (at 218.44 34.29 0)
       (effects (font (size 1.27 1.27)) hide)
     )
