File: SimpleServoTester/SimpleServoTester.kicad_pcb (KiCad board)
At the start: 2 copper layers, 41 parts, among them J1 USBASP, J2 Servo, J3 OLED, Q1 IRLZ44N, SW1 POWER, SW2 SW_Push, U1 ATmega328-A, U2 LM7805_TO220, U3 INA219AxD, U4 AMS1117-3.3, Y2 16MHz

Commit message: update
Parts:
- removed C10: 100n/50V, Capacitor_SMD:C_0603_1608Metric
- removed RV1: 10k, Footprint:PTV09A-4225F-B502
- added C7: 100n/50V, Capacitor_SMD:C_0603_1608Metric, F.Cu at (119.2, 107.5)
- added C8: 100n/50V, Capacitor_SMD:C_0603_1608Metric, F.Cu at (123.8, 107.5)
- added R10: 100R, Resistor_SMD:R_0603_1608Metric, F.Cu at (122.2, 107.5)
- added R8: 100R, Resistor_SMD:R_0603_1608Metric, F.Cu at (120.8, 107.5)
- D1: moved to B.Cu
- H1, H2, H3, H4: footprint MountingHole:MountingHole_3.2mm_M3_Pad_Via -> MountingHole:MountingHole_3.2mm_M3
- J1: moved to F.Cu
- SW2: value SW_Push -> RotaryEncoder_Switch; footprint Footprint:Omron_B3F-12x12mm -> Rotary_Encoder:RotaryEncoder_Alps_EC11E-Switch_Vertical_H20mm
- moved SW2 63.2 mm to (125.2, 119.2), turned to 180 degrees
- moved U4 61.1 mm to (90.5, 70.5), turned to -90 degrees
- moved C11 57.1 mm to (90.8, 64.5)
- moved C13 55.6 mm to (90.8, 60.2)
- moved BT1 54.8 mm to (98.8, 89.8)
- moved C1 54.8 mm to (103.9, 56.8)
- moved C5 54.8 mm to (131.2, 85.5)
- moved J3 54.8 mm to (123.0, 72.5)
- moved L1 54.8 mm to (134.8, 85.3)
- moved R1 54.8 mm to (122.2, 75.8)
- moved U2 54.8 mm to (105.8, 63.0)
- moved C3 54.8 mm to (103.2, 72.5)
- moved Q1 54.8 mm to (105.5, 95.5)
- moved SW1 54.8 mm to (97.5, 46.8)
- moved H1 54.4 mm to (86.2, 47.0)
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Connections:
- U1 pad 1: unconnected-(U1-PD3-Pad1) -> INT_PIN_2
- U1 pad 2: unconnected-(U1-PD4-Pad2) -> DI
Other:
- board outline added: 70.8 x 92.5 mm

Commit message: update
Parts:
- added Q2: S8050, Package_TO_SOT_SMD:SOT-23-3, F.Cu at (131.8, 94.2)
- added R11: 1k, Resistor_SMD:R_0603_1608Metric, F.Cu at (116.8, 92.8)
- added R12: 47k, Resistor_SMD:R_0603_1608Metric, F.Cu at (129.2, 79.5)
- added R13: 47k, Resistor_SMD:R_0603_1608Metric, F.Cu at (129.2, 81.8)
- R7: footprint Resistor_SMD:R_0603_1608Metric -> Resistor_SMD:R_2512_6332Metric
- moved R5 81.0 mm to (92.8, 131.0), turned to 180 degrees
- moved U3 80.9 mm to (99.1, 131.2)
- moved R7 80.7 mm to (105.0, 131.2), turned to -90 degrees
- moved R6 77.7 mm to (92.8, 129.5), turned to 180 degrees
- moved C9 76.9 mm to (99.2, 134.0), turned to 180 degrees
- moved C12 50.3 mm to (140.8, 80.6)
- moved C13 50.3 mm to (141.1, 60.9)
- moved C14 50.3 mm to (141.0, 86.3)
- moved U4 50.3 mm to (140.8, 71.1)
- moved C11 50.3 mm to (141.0, 65.1)
- moved R2 46.7 mm to (101.2, 96.8), turned to -90 degrees
- moved R4 25.2 mm to (117.8, 76.5), turned to -90 degrees
- moved C6 24.2 mm to (125.8, 84.8), turned to 90 degrees
- moved R3 17.1 mm to (120.5, 76.5), turned to -90 degrees
- moved R1 7.29 mm to (115.0, 76.5)
Connections:
- BT1 pad 2: Net-(BT1--) -> AI0
- BT2 pad 1: Net-(BT1--) -> AI0
- U1 pad 11: unconnected-(U1-PD7-Pad11) -> BAT_T
- U1 pad 23: POT -> AI0
- U1 pad 24: unconnected-(U1-PC1-Pad24) -> AI1
Routing:
- net +BATT: track 0.00 -> 20.3 mm
- net /S+: track 0.00 -> 7.08 mm

Commit message: Update SimpleServoTester.kicad_pcb
Parts:
- moved R3 0.25 mm to (120.8, 76.5)
- moved R4 0.25 mm to (118.0, 76.5)
Routing:
- net +5V: track 0.00 -> 106.1 mm
- net AI0: track 0.00 -> 100.7 mm
- net +BATT: track 20.3 -> 99.2 mm
- net SERVO_SIGNAL: track 0.00 -> 62.0 mm
- net Net-(J2-Pin_1): track 0.00 -> 48.1 mm
- net Net-(J2-Pin_2): track 0.00 -> 41.8 mm
- net RESET: track 0.00 -> 29.1 mm
- net +3V3: track 0.00 -> 20.0 mm
- net Net-(R8-Pad2): track 0.00 -> 13.8 mm
- net VDD: track 0.00 -> 12.9 mm
- net Net-(D1-A): track 0.00 -> 12.2 mm
- net SDA: track 0.00 -> 10.3 mm
- net SCL: track 0.00 -> 10.2 mm
- net Net-(R9-Pad1): track 0.00 -> 9.57 mm
- net AI1: track 0.00 -> 8.52 mm
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- added copper zone on B.Cu, net GND
- added copper zone on F.Cu, net GND

Commit message: update
Parts:
- D1: moved to F.Cu
- J1: footprint Connector_IDC:IDC-Header_2x05_P2.54mm_Horizontal -> Connector_PinHeader_2.54mm:PinHeader_1x06_P2.54mm_Horizontal
- moved C9 78.0 mm to (134.3, 64.3), turned to -90 degrees
- moved R7 77.4 mm to (131.6, 58.5), turned to 0 degrees
- moved U3 74.3 mm to (131.5, 64.4), turned to 90 degrees
- moved J2 72.4 mm to (115.5, 53.6), turned to 90 degrees
- moved R5 71.5 mm to (131.3, 70.8), turned to -90 degrees
- moved R6 69.4 mm to (129.8, 70.8), turned to -90 degrees
- moved J1 56.2 mm to (143.5, 104.2), turned to 0 degrees
- moved D1 45.8 mm to (138.8, 102.0), turned to -90 degrees
- moved R2 40.4 mm to (106.0, 56.8), turned to 90 degrees
- moved Q1 34.3 mm to (106.3, 61.2)
- moved C2 18.1 mm to (102.8, 94.8)
- moved C1 18.0 mm to (101.0, 74.5)
- moved L1 17.7 mm to (134.8, 103.0)
- moved R1 17.7 mm to (115.0, 94.2)
- moved R12 17.7 mm to (129.2, 97.2)
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Connections:
- C15 pad 2: INT_PIN -> INT_PIN_2
- C7 pad 2: INT_PIN_2 -> INT_PIN
- J1 pad 1: MOSI -> Net-(D1-A)
- J1 pad 2: Net-(D1-A) -> SCK
- J1 pad 3: unconnected-(J1-Pin_3-Pad3) -> MISO
- J1 pad 4: GND -> MOSI
- R8 pad 1: INT_PIN_2 -> INT_PIN
- R9 pad 2: INT_PIN -> INT_PIN_2
- U1 pad 11: BAT_T -> unconnected-(U1-PD7-Pad11)
- U1 pad 12: unconnected-(U1-PB0-Pad12) -> DI
- U1 pad 2: DI -> GATE_MOSFET
- U1 pad 25: unconnected-(U1-PC2-Pad25) -> BAT_T
- U1 pad 30: GATE_MOSFET -> unconnected-(U1-PD0-Pad30)
Routing:
- net +5V: track 106.1 -> 259.9 mm, vias 0 -> 7
- net SERVO_SIGNAL: track 62.0 -> 142.3 mm, vias 0 -> 3
- net SCL: track 10.2 -> 56.3 mm
- net GATE_MOSFET: track 4.49 -> 49.9 mm
- net +BATT: track 99.2 -> 140.0 mm, vias 0 -> 1
- net SDA: track 10.3 -> 45.0 mm, vias 0 -> 2
- net INT_PIN_2: track 1.53 -> 34.7 mm, vias 0 -> 2
- net +3V3: track 20.0 -> 51.8 mm
- net Net-(J2-Pin_1): track 48.1 -> 16.6 mm
- net INT_PIN: track 1.52 -> 32.2 mm, vias 0 -> 2
- net MOSI: track 0.00 -> 26.3 mm
- net MISO: track 0.00 -> 23.8 mm
- net SCK: track 0.00 -> 21.9 mm
- net DI: track 1.53 -> 16.6 mm
- net RESET: track 29.1 -> 43.9 mm, vias 0 -> 2
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Other:
- board text added: "SWITCH"

Commit message: update
Parts:
- J3: footprint Connector_PinSocket_2.54mm:PinSocket_1x04_P2.54mm_Vertical -> Connector_PinHeader_2.54mm:PinHeader_1x04_P2.54mm_Vertical
- moved R9 4.10 mm to (106.0, 124.5)
- moved C15 3.72 mm to (106.0, 122.5)
- moved C7 3.36 mm to (106.0, 120.5)
- moved Q2 3.21 mm to (129.2, 90.5)
- moved R11 3.20 mm to (125.2, 94.0)
- moved R12 3.20 mm to (129.2, 94.0)
- moved R13 3.17 mm to (129.2, 96.3)
- moved R8 3.03 mm to (106.0, 118.5)
- moved R10 2.77 mm to (106.0, 116.5)
- moved C8 2.61 mm to (106.0, 114.5)
- moved C2 2.47 mm to (101.0, 93.0)
- moved L1 2.00 mm to (133.0, 104.0)
- moved C5 1.91 mm to (129.5, 104.0)
- moved C13 1.00 mm to (144.5, 56.2)
- moved R6 0.80 mm to (129.0, 70.8)
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Routing:
- net +5V: track 259.9 -> 207.5 mm, vias 7 -> 6
- net SERVO_SIGNAL: track 142.3 -> 155.2 mm, vias 3 -> 1
- net GATE_MOSFET: track 49.9 -> 59.8 mm
- net INT_PIN_2: track 34.7 -> 41.1 mm
- net INT_PIN: track 32.2 -> 38.2 mm
- net SCL: track 56.3 -> 50.7 mm, vias 0 -> 2
- net GND: track 14.0 -> 9.92 mm, vias 3 -> 1
- net RESET: track 43.9 -> 39.8 mm
- net +BATT: track 140.0 -> 136.8 mm, vias 1 -> 2
- net Net-(R8-Pad2): track 14.5 -> 17.6 mm
- net Net-(R10-Pad2): track 7.44 -> 10.4 mm
- net DI: track 16.6 -> 19.3 mm
- net SDA: track 45.0 -> 42.3 mm
- net BAT_T: track 4.04 -> 6.24 mm
- net AI1: track 8.52 -> 10.4 mm
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Other:
- board text added: "+5V"
- board text added: "GND"
- board text added: "SIGNAL"

Commit message: update
Parts:
- moved C3 4.35 mm to (101.0, 83.2), turned to 90 degrees
- moved Q1 3.54 mm to (105.8, 64.7)
- moved R2 3.50 mm to (106.2, 60.2)
- moved U2 2.05 mm to (105.8, 76.4)
- moved C1 0.50 mm to (101.0, 75.0), turned to -90 degrees
Routing:
- net +5V: track 207.5 -> 311.5 mm, vias 6 -> 21
- net GND: track 9.92 -> 17.0 mm
- net Net-(J2-Pin_1): track 15.4 -> 19.1 mm
- net GATE_MOSFET: track 59.8 -> 58.0 mm, vias 0 -> 1
- net +3V3: track 53.4 -> 52.0 mm
- net SERVO_SIGNAL: track 155.2 -> 156.4 mm
- net +BATT: track 136.8 -> 137.9 mm
- net Net-(J2-Pin_2): track 30.9 -> 30.1 mm
- added copper zone on B.Cu, net +5V
- added copper zone on F.Cu, net +5V
Other:
- outline, holes or cut-outs redrawn
- board text added: "3V3"
- board text added: "7805"
- board text added: "IRLZ44N"
- board text added: "MISO"
- board text added: "MOSI"
- board text added: "RESET"
- board text added: "SCK"
- board text added: "SCL"
- board text added: "SDA"

Commit message: Initial release
Parts:
- added G***: LOGO, Footprint:tvz2, F.Cu at (90.2, 68.5)
Other:
- board text added: "JLCJLCJLCJLC"
- board text added: "SimpleServoTesterV1rev1"
